File: SnapICSP/SnapICSP.sch (KiCad schematic (older format))
At the start: 3 parts, among them J1 Conn_01x08_Male, J2 AVR-ISP-6, J3 AVR-ISP-6

Commit message: Corrected pinout on component
Parts:
- J1: footprint Socket_Strips:Socket_Strip_Straight_1x08_Pitch2.54mm -> Pin_Headers:Pin_Header_Angled_1x08_Pitch2.54mm
- J2: footprint Socket_Strips:Socket_Strip_Straight_2x03_Pitch2.00mm -> Pin_Headers:Pin_Header_Straight_2x03_Pitch2.00mm
- J3: footprint Socket_Strips:Socket_Strip_Straight_2x03_Pitch2.54mm -> Pin_Headers:Pin_Header_Straight_2x03_Pitch2.54mm
Changed lines of the file:
@@
 F 0 "J2" H 2325 3350 50  0000 R CNN
 F 1 "AVR-ISP-6" H 2475 2550 50  0000 R CNN
-F 2 "Socket_Strips:Socket_Strip_Straight_2x03_Pitch2.00mm" V 1800 2950 50  0001 C CNN
+F 2 "Pin_Headers:Pin_Header_Straight_2x03_Pitch2.00mm" V 1800 2950 50  0001 C CNN
 F 3 " ~" H 775 2350 50  0001 C CNN
 	1    2050 2900
@@
 F 0 "J3" H 4000 3350 50  0000 R CNN
 F 1 "AVR-ISP-6" H 4150 2550 50  0000 R CNN
-F 2 "Socket_Strips:Socket_Strip_Straight_2x03_Pitch2.54mm" V 3450 2950 50  0001 C CNN
+F 2 "Pin_Headers:Pin_Header_Straight_2x03_Pitch2.54mm" V 3450 2950 50  0001 C CNN
 F 3 " ~" H 2425 2350 50  0001 C CNN
 	1    3700 2900
@@
 F 0 "J1" H 1750 1725 50  0000 C CNN
 F 1 "Conn_01x08_Male" H 1750 875 50  0000 C CNN
-F 2 "Socket_Strips:Socket_Strip_Straight_1x08_Pitch2.54mm" H 1750 1350 50  0001 C CNN
+F 2 "Pin_Headers:Pin_Header_Angled_1x08_Pitch2.54mm" H 1750 1350 50  0001 C CNN
 F 3 "~" H 1750 1350 50  0001 C CNN
 	1    1750 1350
